File: untitled.sch (EAGLE design)
At the start: 7 parts, among them U1 EFM8SB20F16G-A-QFN24QFN24_4X4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, U2 LTC3106EFE#PBF

Commit message: Check in
Parts:
- added C4: 47uF, SparkFun-Capacitors:4.7UF0603
- added C5: 10uF, SparkFun-Capacitors:10UF-0603-6.3V-20%
- added C6, C7, C8: 0.1uF, SparkFun-Capacitors:0.1UF-0603-25V-(+80/-20%)
- added J1: (no value), SparkFun-Connectors:CONN_023.5MM
- added Q1: 2.5A/30V/105mΩ, SparkFun-DiscreteSemi:MOSFET_PCH-DMG2307L
- added R1: 2.0M, SparkFun-Resistors:2MOHMS-0603-1/10W-1%
- added R2: 365k, SparkFun-Resistors:390KOHM-0603-1/10W-1%
- added U3: EFM8SB10F8G-A-QFN24QFN24_4X4-M, EFM8SB10F8A-A-QFN24:EFM8SB10F8G-A-QFN24QFN24_4X4-M
- added U4: RFM95W-915S2, RFM95W-915S2:RFM95W-915S2
- C3: value 4.7uF -> 47uF
- U1: value EFM8SB20F16G-A-QFN24QFN24_4X4-M -> TS3A4751PWR; device EFM8_BusyBee:EFM8SB20F16G-A-QFN24QFN24_4X4-M -> TS3A4751PWR:TS3A4751PWR
Connections:
- new net N$4: BATT1.+, Q1.D
- new net N$5: R1.1, R2.2, U2.RUN
- new net VCC_1: C8.2, U1.NO1, U4.3.3V
- new net VIN: C5.1, J1.2, R1.2, U2.VIN
- new net V_BATT: C4.2, Q1.S, U2.ENVSTR, U2.VCAP, U2.VSTORE
- net 3.3V: now also C3.1, C6.1, C7.1, U1.COM1, U1.VCC, U3.VDD/VIO
- net CS: now also U3.P0.5, U4.NSS; no longer U1.P1.3
- net GND: now also BATT1.-, C3.2, C4.1, C5.2, C6.2, C7.2, C8.1, J1.1, Q1.G, R2.1, U3.GND, U3.GND_2, U4.GND; no longer U1.GND_2
- net MISO: now also U3.P0.1, U4.MISO; no longer U1.P1.1
- net MOSI: now also U3.P0.2, U4.MOSI; no longer U1.P1.2
- net SCK: now also U3.P0.0, U4.SCK; no longer U1.P1.0
- net SCL: now also U3.P0.4; no longer U1.P0.1
- net SDA: now also U3.P0.3; no longer U1.P0.0
