File: STM32LoRa.brd (EAGLE design)
At the start: 57 x 106.8 mm, 40 parts, among them IC1 CMWX1ZZABZ-078, J3 USB_MINI-B_SMT, J4 Qwiic Right Angle, J7 U.FL, Q1 2.5A/30V/105mΩ, U1 TS3A4751PWR, U2 LTC3106EFE#PBF

Commit message: File check in
Parts:
- removed J3: USB_MINI-B_SMT, SparkFun-Connectors:USB-MINIB
- added C16, C17: 0.1uF, SparkFun-Capacitors:0603
- added J8: USB3131-30-0230-A_REVB, USB3131-30-0230-A_REVB:GCT_USB3131-30-0230-A_REVB
- moved S2 213.9 mm to (46.9, 41.7), turned to 270 degrees
- moved D1 200.3 mm to (19.9, 92.5)
- moved C14 189.2 mm to (47.0, 30.5)
- moved R7 188.5 mm to (15.0, 12.2), turned to 270 degrees
- moved D3 186.8 mm to (34.8, 19.7), turned to 270 degrees
- moved R4 186.7 mm to (36.4, 37.3), turned to 270 degrees
- moved R5 186.3 mm to (34.8, 15.0), turned to 270 degrees
- moved C15 185.8 mm to (32.5, 37.1), turned to 270 degrees
- moved R6 184.5 mm to (13.1, 12.2), turned to 270 degrees
- moved J5 180.2 mm to (5.21, 18.3), turned to 270 degrees
- moved J4 178.0 mm to (6.73, 23.7), turned to 270 degrees
- moved C13 167.2 mm to (24.6, 28.2), turned to 270 degrees
- moved C6 165.4 mm to (47.0, 32.1)
- moved R3 164.8 mm to (23.9, 37.7), turned to 270 degrees
- moved C12 163.8 mm to (23.1, 28.2), turned to 90 degrees
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Connections:
- removed net N$7: J3.ID, R3.2
- removed net V_USB: D2.A, J3.VBUS
- new net N$12: J8.4, R3.2
- new net N$13: D2.A, J8.1
- net GND: now also C16.1, C17.1, J8.5, J8.S1, J8.S2; no longer J3.GND, J3.S1, J3.S2, J3.S3, J3.S4
- net USB_N: now also J8.2; no longer J3.D-
- net USB_P: now also J8.3; no longer J3.D+
- net VCC_1: now also C16.2, C17.2
Routing:
- net 3.3V: track 0.00 -> 213.8 mm, vias 0 -> 3
- net VIN: track 0.00 -> 88.1 mm
- net V_BATT: track 0.00 -> 65.8 mm, vias 0 -> 3
- net VCC_1: track 0.00 -> 63.8 mm, vias 0 -> 2
- net SCL_IN: track 0.00 -> 52.4 mm, vias 0 -> 2
- net SDA_IN: track 0.00 -> 48.5 mm, vias 0 -> 2
- net SWITCH_EN: track 0.00 -> 45.2 mm
- net SDA_OUT: track 0.00 -> 35.2 mm, vias 0 -> 2
- net VCC: track 0.00 -> 28.5 mm
- net SCL_OUT: track 0.00 -> 25.7 mm
- net !NRST: track 0.00 -> 24.6 mm
- net N$8: track 0.00 -> 21.2 mm, vias 0 -> 2
- net SWCLK: track 0.00 -> 18.2 mm
- net SWDIO: track 0.00 -> 13.2 mm
- net USB_P: track 0.00 -> 12.0 mm
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- added copper zone on layer 1, net GND
- added copper zone on layer 16, net GND
- added copper zone on layer 1, net N$4
